File: pyaa.sch (KiCad schematic (older format))
At the start: 18 parts, among them J1 MJ-4PP-9, K0 KEYSW, K1 KEYSW, SW1 SW_PUSH, U1 ProMicro

Commit message: Add files via upload
Parts:
- U1: footprint Keebio-Parts:ArduinoProMicro -> Lily58-footprint:ProMicro_rev2
Connections:
- wire segments 53 -> 54
Other:
- moved on the sheet: K0, K1, KA1, KKL1, KN1, KO1, KPL1, KS1, KS2, KST1, KTL1, KWL1
