File: pyaa.sch (KiCad schematic (older format))
At the start: 18 parts, among them J1 MJ-4PP-9, K0 KEYSW, K1 KEYSW, SW1 SW_PUSH, U1 ProMicro

Commit message: update files
Parts:
- added J2: MJ-4PP-9, Keebio-Parts:TRRS-PJ-320A, symbol Connector:AudioJack4
- added KBR1, KDR1, KER1, KFR1, KGR1, KLR1, KN2, KPR1, KRR1, KSR1, KST3, KST4, KTR1, KUR1, KZR1: KEYSW, switches:Choc_PG1350_Choc_Spacing, symbol keyboard_parts:KEYSW
- added SW2: SW_PUSH, Lily58-footprint:TACT_SWITCH_TVBP06, symbol keyboard_parts:SW_PUSH
- added U2: ProMicro, Lily58-footprint:ProMicro_rev, symbol promicro:ProMicro
- J1: footprint Lily58_Footprints:MJ-4PP-9_rev2 -> Keebio-Parts:TRRS-PJ-320A; symbol mj-4pp-9:MJ-4PP-9 -> Connector:AudioJack4
- K0, K1, KA1, KHL1, KKL1, KN1, KO1, KPL1, KRL1, KST1, KST2, KTL1, KWL1: footprint switches:Choc_PG1350_Choc_Spacing_Reversible -> switches:Choc_PG1350_Choc_Spacing
- KSL1: renamed from KS1; footprint switches:Choc_PG1350_Choc_Spacing_Reversible -> switches:Choc_PG1350_Choc_Spacing
- KSL2: renamed from KS2; footprint switches:Choc_PG1350_Choc_Spacing_Reversible -> switches:Choc_PG1350_Choc_Spacing
- U1: footprint Keebio-Parts:ArduinoProMicro -> Lily58-footprint:ProMicro_rev
Connections:
- wire segments 53 -> 110
- no-connect marks 5 -> 9
Other:
- moved on the sheet: K0, K1, KA1, KHL1, KKL1, KN1, KO1, KPL1, KRL1, KSL1, KSL2, KST1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
