File: pyaa.kicad_pcb (KiCad board)
At the start: 2 copper layers, 123 x 80.1 mm, 18 parts, among them J1 MJ-4PP-9, K0 KEYSW, K1 KEYSW, SW1 SW_PUSH, U1 ProMicro

Commit message: Add files via upload
Parts:
- U1: footprint Keebio-Parts:ArduinoProMicro -> Lily58-footprint:ProMicro_rev2
- moved U1 22.3 mm to (101.5, 91.0), turned to 0 degrees
- moved KN1 21.9 mm to (138.7, 123.7)
- moved K0 21.9 mm to (207.2, 82.3)
- moved K1 21.9 mm to (207.2, 100.3)
- moved KA1 21.9 mm to (121.0, 126.8)
- moved KHL1 21.9 mm to (136.2, 75.2)
- moved KKL1 21.9 mm to (172.2, 93.2)
- moved KO1 21.9 mm to (103.3, 129.9)
- moved KPL1 21.9 mm to (154.2, 70.8)
- moved KRL1 21.9 mm to (136.2, 93.2)
- moved KS1 21.9 mm to (190.2, 82.3)
- moved KS2 21.9 mm to (190.2, 100.3)
- moved KST1 21.9 mm to (119.2, 75.2)
- moved KST2 21.9 mm to (119.2, 93.2)
- moved KTL1 21.9 mm to (172.2, 75.2)
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Routing:
- net Net-(J1-PadB): track 28.8 -> 59.7 mm, vias 0 -> 1
- net VDD: track 33.1 -> 55.0 mm
- net Net-(KO1-Pad1): track 28.5 -> 49.0 mm, vias 0 -> 1
- net Net-(KKL1-Pad1): track 114.0 -> 134.3 mm, vias 0 -> 1
- net Net-(KWL1-Pad1): track 86.5 -> 106.6 mm, vias 0 -> 1
- net Net-(KS2-Pad1): track 138.8 -> 159.0 mm, vias 0 -> 1
- net Net-(KRL1-Pad1): track 68.0 -> 88.0 mm, vias 0 -> 1
- net Net-(KA1-Pad1): track 47.4 -> 67.1 mm, vias 0 -> 1
- net Net-(KN1-Pad1): track 68.1 -> 87.6 mm, vias 0 -> 1
- net Net-(KST1-Pad1): track 35.5 -> 53.0 mm
- net Net-(KST2-Pad1): track 8.76 -> 23.8 mm
- net Net-(KHL1-Pad1): track 27.2 -> 41.4 mm
- net Net-(KS1-Pad1): track 88.4 -> 102.6 mm
- net Net-(KPL1-Pad1): track 53.9 -> 68.1 mm
- net Net-(K0-Pad1): track 113.5 -> 127.7 mm
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- added copper zone on B.Cu, net (none)
Other:
- board size 123 x 80.1 mm -> 123.4 x 80.1 mm

Commit message: Add files via upload
Parts:
- moved SW1 0.66 mm to (107.9, 113.0)
- moved J1 0.60 mm to (91.6, 112.0)
- moved KA1 0.32 mm to (120.7, 126.8)
- moved KN1 0.32 mm to (138.4, 123.7)
- moved KO1 0.32 mm to (103.0, 129.9)
Connections:
- U1 pad 1: Net-(U1-Pad1) -> Net-(J1-PadB)
- U1 pad 10: Net-(KO1-Pad1) -> Net-(U1-Pad10)
- U1 pad 11: Net-(KA1-Pad1) -> Net-(U1-Pad11)
- U1 pad 12: Net-(KN1-Pad1) -> Net-(KA1-Pad1)
- U1 pad 13: Net-(KST1-Pad1) -> Net-(KN1-Pad1)
- U1 pad 14: Net-(K1-Pad1) -> Net-(KO1-Pad1)
- U1 pad 16: Net-(K0-Pad1) -> Net-(KWL1-Pad1)
- U1 pad 17: Net-(KS1-Pad1) -> Net-(KS2-Pad1)
- U1 pad 18: Net-(KTL1-Pad1) -> Net-(K0-Pad1)
- U1 pad 19: Net-(KPL1-Pad1) -> Net-(KTL1-Pad1)
- U1 pad 2: Net-(U1-Pad2) -> Net-(KST1-Pad1)
- U1 pad 5: Net-(J1-PadB) -> Net-(KPL1-Pad1)
- U1 pad 6: Net-(KS2-Pad1) -> Net-(KS1-Pad1)
- U1 pad 7: Net-(KKL1-Pad1) -> Net-(K1-Pad1)
- U1 pad 8: Net-(KWL1-Pad1) -> Net-(KKL1-Pad1)
Routing:
- net Net-(KS2-Pad1): track 159.0 -> 110.2 mm, vias 1 -> 0
- net Net-(KKL1-Pad1): track 134.3 -> 89.2 mm, vias 1 -> 0
- net Net-(KWL1-Pad1): track 106.6 -> 63.4 mm, vias 1 -> 0
- net Net-(KRL1-Pad1): track 88.0 -> 48.9 mm, vias 1 -> 0
- net Net-(KST1-Pad1): track 53.0 -> 23.4 mm
- net Net-(J1-PadB): track 59.7 -> 83.4 mm, vias 1 -> 0
- net Net-(K1-Pad1): track 135.7 -> 124.4 mm
- net Net-(KO1-Pad1): track 49.0 -> 39.7 mm, vias 1 -> 0
- net Net-(KN1-Pad1): track 87.6 -> 81.3 mm, vias 1 -> 0
- net GND: track 17.2 -> 11.3 mm
- net Net-(K0-Pad1): track 127.7 -> 122.6 mm
- net Net-(KS1-Pad1): track 102.6 -> 99.9 mm
- net Net-(KTL1-Pad1): track 81.7 -> 79.2 mm
- net Net-(KA1-Pad1): track 67.1 -> 65.7 mm, vias 1 -> 0
- net Net-(SW1-Pad1): track 47.0 -> 46.4 mm
- removed copper zone on B.Cu, net (none)
Other:
- board size 123.4 x 80.1 mm -> 123.5 x 80.1 mm
